Commit message: Change description to be comppatible with ROS2 jazzy

File: urdf/aubo_C10.urdf (robot description, URDF)
Before this commit: robot aubo_C10, 8 links, 7 joints
Links:
- link base_link: geometry collision mesh filename=file://$(find aubo_description)/meshes/aubo_C10/collision/l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; visual mesh filename=file://$(find aubo_description)/meshes/aubo_C10/visual/link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
- link foreArm_Link: geometry collision mesh filename=file://$(find aubo_description)/meshes/aubo_C10/collision/l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; visual mesh filename=file://$(find aubo_description)/meshes/aubo_C10/visual/link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
- link shoulder_Link: geometry collision mesh filename=file://$(find aubo_description)/meshes/aubo_C10/collision/l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; visual mesh filename=file://$(find aubo_description)/meshes/aubo_C10/visual/link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
- link upperArm_Link: geometry collision mesh filename=file://$(find aubo_description)/meshes/aubo_C10/collision/l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; visual mesh filename=file://$(find aubo_description)/meshes/aubo_C10/visual/link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
- link wrist1_Link: geometry collision mesh filename=file://$(find aubo_description)/meshes/aubo_C10/collision/l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; visual mesh filename=file://$(find aubo_description)/meshes/aubo_C10/visual/link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
- link wrist2_Link: geometry collision mesh filename=file://$(find aubo_description)/meshes/aubo_C10/collision/l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; visual mesh filename=file://$(find aubo_description)/meshes/aubo_C10/visual/link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
- link wrist3_Link: geometry collision mesh filename=file://$(find aubo_description)/meshes/aubo_C10/collision/l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; visual mesh filename=file://$(find aubo_description)/meshes/aubo_C10/visual/link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

File: urdf/aubo_C16_30.urdf (robot description, URDF)
Before this commit: robot aubo_C16_30, 8 links, 7 joints
Links:
- link base_link: geometry collision mesh filename=file://$(find aubo_description)/meshes/aubo_C16_30/collisio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; visual mesh filename=file://$(find aubo_description)/meshes/aubo_C16_30/visual/l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
- link foreArm_Link: geometry collision mesh filename=file://$(find aubo_description)/meshes/aubo_C16_30/collisio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; visual mesh filename=file://$(find aubo_description)/meshes/aubo_C16_30/visual/l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
- link shoulder_Link: geometry collision mesh filename=file://$(find aubo_description)/meshes/aubo_C16_30/collisio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; visual mesh filename=file://$(find aubo_description)/meshes/aubo_C16_30/visual/l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
- link upperArm_Link: geometry collision mesh filename=file://$(find aubo_description)/meshes/aubo_C16_30/collisio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; visual mesh filename=file://$(find aubo_description)/meshes/aubo_C16_30/visual/l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
- link wrist1_Link: geometry collision mesh filename=file://$(find aubo_description)/meshes/aubo_C16_30/collisio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; visual mesh filename=file://$(find aubo_description)/meshes/aubo_C16_30/visual/l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
- link wrist2_Link: geometry collision mesh filename=file://$(find aubo_description)/meshes/aubo_C16_30/collisio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; visual mesh filename=file://$(find aubo_description)/meshes/aubo_C16_30/visual/l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
- link wrist3_Link: geometry collision mesh filename=file://$(find aubo_description)/meshes/aubo_C16_30/collisio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; visual mesh filename=file://$(find aubo_description)/meshes/aubo_C16_30/visual/l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

File: urdf/aubo_C20_30.urdf (robot description, URDF)
Before this commit: robot aubo_C20_30, 8 links, 7 joints
Links:
- link base_link: geometry collision mesh filename=file://$(find aubo_description)/meshes/aubo_C20_30/collisio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; visual mesh filename=file://$(find aubo_description)/meshes/aubo_C20_30/visual/l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
- link foreArm_Link: geometry collision mesh filename=file://$(find aubo_description)/meshes/aubo_C20_30/collisio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; visual mesh filename=file://$(find aubo_description)/meshes/aubo_C20_30/visual/l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
- link shoulder_Link: geometry collision mesh filename=file://$(find aubo_description)/meshes/aubo_C20_30/collisio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; visual mesh filename=file://$(find aubo_description)/meshes/aubo_C20_30/visual/l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
- link upperArm_Link: geometry collision mesh filename=file://$(find aubo_description)/meshes/aubo_C20_30/collisio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; visual mesh filename=file://$(find aubo_description)/meshes/aubo_C20_30/visual/l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
- link wrist1_Link: geometry collision mesh filename=file://$(find aubo_description)/meshes/aubo_C20_30/collisio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; visual mesh filename=file://$(find aubo_description)/meshes/aubo_C20_30/visual/l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
- link wrist2_Link: geometry collision mesh filename=file://$(find aubo_description)/meshes/aubo_C20_30/collisio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; visual mesh filename=file://$(find aubo_description)/meshes/aubo_C20_30/visual/l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
- link wrist3_Link: geometry collision mesh filename=file://$(find aubo_description)/meshes/aubo_C20_30/collisio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; visual mesh filename=file://$(find aubo_description)/meshes/aubo_C20_30/visual/l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

File: urdf/aubo_C3.urdf (robot description, URDF)
Before this commit: robot aubo_C3, 8 links, 7 joints
Links:
- link base_link: geometry collision mesh filename=file://$(find aubo_description)/meshes/aubo_C3/collision/li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; visual mesh filename=file://$(find aubo_description)/meshes/aubo_C3/visual/link0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
- link foreArm_Link: geometry collision mesh filename=file://$(find aubo_description)/meshes/aubo_C3/collision/li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; visual mesh filename=file://$(find aubo_description)/meshes/aubo_C3/visual/link3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
- link shoulder_Link: geometry collision mesh filename=file://$(find aubo_description)/meshes/aubo_C3/collision/li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; visual mesh filename=file://$(find aubo_description)/meshes/aubo_C3/visual/link1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
- link upperArm_Link: geometry collision mesh filename=file://$(find aubo_description)/meshes/aubo_C3/collision/li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; visual mesh filename=file://$(find aubo_description)/meshes/aubo_C3/visual/link2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
- link wrist1_Link: geometry collision mesh filename=file://$(find aubo_description)/meshes/aubo_C3/collision/li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; visual mesh filename=file://$(find aubo_description)/meshes/aubo_C3/visual/link4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
- link wrist2_Link: geometry collision mesh filename=file://$(find aubo_description)/meshes/aubo_C3/collision/li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; visual mesh filename=file://$(find aubo_description)/meshes/aubo_C3/visual/link5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
- link wrist3_Link: geometry collision mesh filename=file://$(find aubo_description)/meshes/aubo_C3/collision/li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; visual mesh filename=file://$(find aubo_description)/meshes/aubo_C3/visual/link6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

File: urdf/aubo_C3_30.urdf (robot description, URDF)
Before this commit: robot aubo_C3_30, 8 links, 7 joints
Links:
- link base_link: geometry collision mesh filename=file://$(find aubo_description)/meshes/aubo_C3_30/collision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; visual mesh filename=file://$(find aubo_description)/meshes/aubo_C3_30/visual/li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
- link foreArm_Link: geometry collision mesh filename=file://$(find aubo_description)/meshes/aubo_C3_30/collision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; visual mesh filename=file://$(find aubo_description)/meshes/aubo_C3_30/visual/li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
- link shoulder_Link: geometry collision mesh filename=file://$(find aubo_description)/meshes/aubo_C3_30/collision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; visual mesh filename=file://$(find aubo_description)/meshes/aubo_C3_30/visual/li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
- link upperArm_Link: geometry collision mesh filename=file://$(find aubo_description)/meshes/aubo_C3_30/collision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; visual mesh filename=file://$(find aubo_description)/meshes/aubo_C3_30/visual/li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
- link wrist1_Link: geometry collision mesh filename=file://$(find aubo_description)/meshes/aubo_C3_30/collision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; visual mesh filename=file://$(find aubo_description)/meshes/aubo_C3_30/visual/li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
- link wrist2_Link: geometry collision mesh filename=file://$(find aubo_description)/meshes/aubo_C3_30/collision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; visual mesh filename=file://$(find aubo_description)/meshes/aubo_C3_30/visual/li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
- link wrist3_Link: geometry collision mesh filename=file://$(find aubo_description)/meshes/aubo_C3_30/collision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; visual mesh filename=file://$(find aubo_description)/meshes/aubo_C3_30/visual/li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

File: urdf/aubo_C3_39.urdf (robot description, URDF)
Before this commit: robot aubo_C3_39, 8 links, 7 joints
Links:
- link base_link: geometry collision mesh filename=file://$(find aubo_description)/meshes/aubo_C3_39/collision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; visual mesh filename=file://$(find aubo_description)/meshes/aubo_C3_39/visual/li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
- link foreArm_Link: geometry collision mesh filename=file://$(find aubo_description)/meshes/aubo_C3_39/collision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; visual mesh filename=file://$(find aubo_description)/meshes/aubo_C3_39/visual/li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
- link shoulder_Link: geometry collision mesh filename=file://$(find aubo_description)/meshes/aubo_C3_39/collision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; visual mesh filename=file://$(find aubo_description)/meshes/aubo_C3_39/visual/li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
- link upperArm_Link: geometry collision mesh filename=file://$(find aubo_description)/meshes/aubo_C3_39/collision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; visual mesh filename=file://$(find aubo_description)/meshes/aubo_C3_39/visual/li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
- link wrist1_Link: geometry collision mesh filename=file://$(find aubo_description)/meshes/aubo_C3_39/collision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; visual mesh filename=file://$(find aubo_description)/meshes/aubo_C3_39/visual/li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
- link wrist2_Link: geometry collision mesh filename=file://$(find aubo_description)/meshes/aubo_C3_39/collision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; visual mesh filename=file://$(find aubo_description)/meshes/aubo_C3_39/visual/li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
- link wrist3_Link: geometry collision mesh filename=file://$(find aubo_description)/meshes/aubo_C3_39/collision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; visual mesh filename=file://$(find aubo_description)/meshes/aubo_C3_39/visual/li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

File: urdf/aubo_C5.urdf (robot description, URDF)
Before this commit: robot aubo_C5, 8 links, 7 joints
Links:
- link base_link: geometry collision mesh filename=file://$(find aubo_description)/meshes/aubo_C5/collision/li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; visual mesh filename=file://$(find aubo_description)/meshes/aubo_C5/visual/link0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
- link foreArm_Link: geometry collision mesh filename=file://$(find aubo_description)/meshes/aubo_C5/collision/li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; visual mesh filename=file://$(find aubo_description)/meshes/aubo_C5/visual/link3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
- link shoulder_Link: geometry collision mesh filename=file://$(find aubo_description)/meshes/aubo_C5/collision/li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; visual mesh filename=file://$(find aubo_description)/meshes/aubo_C5/visual/link1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
- link upperArm_Link: geometry collision mesh filename=file://$(find aubo_description)/meshes/aubo_C5/collision/li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; visual mesh filename=file://$(find aubo_description)/meshes/aubo_C5/visual/link2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
- link wrist1_Link: geometry collision mesh filename=file://$(find aubo_description)/meshes/aubo_C5/collision/li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; visual mesh filename=file://$(find aubo_description)/meshes/aubo_C5/visual/link4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
- link wrist2_Link: geometry collision mesh filename=file://$(find aubo_description)/meshes/aubo_C5/collision/li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; visual mesh filename=file://$(find aubo_description)/meshes/aubo_C5/visual/link5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
- link wrist3_Link: geometry collision mesh filename=file://$(find aubo_description)/meshes/aubo_C5/collision/li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; visual mesh filename=file://$(find aubo_description)/meshes/aubo_C5/visual/link6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

File: urdf/aubo_C5_30.urdf (robot description, URDF)
Before this commit: robot aubo_C5_30, 8 links, 7 joints
Links:
- link base_link: geometry collision mesh filename=file://$(find aubo_description)/meshes/aubo_C5_30/collision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; visual mesh filename=file://$(find aubo_description)/meshes/aubo_C5_30/visual/li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
- link foreArm_Link: geometry collision mesh filename=file://$(find aubo_description)/meshes/aubo_C5_30/collision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; visual mesh filename=file://$(find aubo_description)/meshes/aubo_C5_30/visual/li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
- link shoulder_Link: geometry collision mesh filename=file://$(find aubo_description)/meshes/aubo_C5_30/collision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; visual mesh filename=file://$(find aubo_description)/meshes/aubo_C5_30/visual/li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
- link upperArm_Link: geometry collision mesh filename=file://$(find aubo_description)/meshes/aubo_C5_30/collision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; visual mesh filename=file://$(find aubo_description)/meshes/aubo_C5_30/visual/li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
- link wrist1_Link: geometry collision mesh filename=file://$(find aubo_description)/meshes/aubo_C5_30/collision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; visual mesh filename=file://$(find aubo_description)/meshes/aubo_C5_30/visual/li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
- link wrist2_Link: geometry collision mesh filename=file://$(find aubo_description)/meshes/aubo_C5_30/collision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; visual mesh filename=file://$(find aubo_description)/meshes/aubo_C5_30/visual/li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
- link wrist3_Link: geometry collision mesh filename=file://$(find aubo_description)/meshes/aubo_C5_30/collision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; visual mesh filename=file://$(find aubo_description)/meshes/aubo_C5_30/visual/li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

File: urdf/aubo_C5_39.urdf (robot description, URDF)
Before this commit: robot aubo_C5_39, 8 links, 7 joints
Links:
- link base_link: geometry collision mesh filename=file://$(find aubo_description)/meshes/aubo_C5_39/collision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; visual mesh filename=file://$(find aubo_description)/meshes/aubo_C5_39/visual/li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
- link foreArm_Link: geometry collision mesh filename=file://$(find aubo_description)/meshes/aubo_C5_39/collision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; visual mesh filename=file://$(find aubo_description)/meshes/aubo_C5_39/visual/li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
- link shoulder_Link: geometry collision mesh filename=file://$(find aubo_description)/meshes/aubo_C5_39/collision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; visual mesh filename=file://$(find aubo_description)/meshes/aubo_C5_39/visual/li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
- link upperArm_Link: geometry collision mesh filename=file://$(find aubo_description)/meshes/aubo_C5_39/collision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; visual mesh filename=file://$(find aubo_description)/meshes/aubo_C5_39/visual/li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
- link wrist1_Link: geometry collision mesh filename=file://$(find aubo_description)/meshes/aubo_C5_39/collision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; visual mesh filename=file://$(find aubo_description)/meshes/aubo_C5_39/visual/li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
- link wrist2_Link: geometry collision mesh filename=file://$(find aubo_description)/meshes/aubo_C5_39/collision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; visual mesh filename=file://$(find aubo_description)/meshes/aubo_C5_39/visual/li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
- link wrist3_Link: geometry collision mesh filename=file://$(find aubo_description)/meshes/aubo_C5_39/collision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; visual mesh filename=file://$(find aubo_description)/meshes/aubo_C5_39/visual/li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

File: urdf/aubo_E10.urdf (robot description, URDF)
Before this commit: robot aubo_E10, 8 links, 7 joints
Links:
- link base_link: geometry collision mesh filename=file://$(find aubo_description)/meshes/aubo_E10/collision/l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; visual mesh filename=file://$(find aubo_description)/meshes/aubo_E10/visual/link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
- link foreArm_Link: geometry collision mesh filename=file://$(find aubo_description)/meshes/aubo_E10/collision/l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; visual mesh filename=file://$(find aubo_description)/meshes/aubo_E10/visual/link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
- link shoulder_Link: geometry collision mesh filename=file://$(find aubo_description)/meshes/aubo_E10/collision/l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; visual mesh filename=file://$(find aubo_description)/meshes/aubo_E10/visual/link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
- link upperArm_Link: geometry collision mesh filename=file://$(find aubo_description)/meshes/aubo_E10/collision/l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; visual mesh filename=file://$(find aubo_description)/meshes/aubo_E10/visual/link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
- link wrist1_Link: geometry collision mesh filename=file://$(find aubo_description)/meshes/aubo_E10/collision/l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; visual mesh filename=file://$(find aubo_description)/meshes/aubo_E10/visual/link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
- link wrist2_Link: geometry collision mesh filename=file://$(find aubo_description)/meshes/aubo_E10/collision/l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; visual mesh filename=file://$(find aubo_description)/meshes/aubo_E10/visual/link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
- link wrist3_Link: geometry collision mesh filename=file://$(find aubo_description)/meshes/aubo_E10/collision/l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; visual mesh filename=file://$(find aubo_description)/meshes/aubo_E10/visual/link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

File: urdf/aubo_E10_10.urdf (robot description, URDF)
Before this commit: robot aubo_E10_10, 8 links, 7 joints
Links:
- link base_link: geometry collision mesh filename=file://$(find aubo_description)/meshes/aubo_E10_10/collisio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; visual mesh filename=file://$(find aubo_description)/meshes/aubo_E10_10/visual/l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
- link foreArm_Link: geometry collision mesh filename=file://$(find aubo_description)/meshes/aubo_E10_10/collisio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; visual mesh filename=file://$(find aubo_description)/meshes/aubo_E10_10/visual/l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
- link shoulder_Link: geometry collision mesh filename=file://$(find aubo_description)/meshes/aubo_E10_10/collisio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; visual mesh filename=file://$(find aubo_description)/meshes/aubo_E10_10/visual/l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
- link upperArm_Link: geometry collision mesh filename=file://$(find aubo_description)/meshes/aubo_E10_10/collisio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; visual mesh filename=file://$(find aubo_description)/meshes/aubo_E10_10/visual/l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
- link wrist1_Link: geometry collision mesh filename=file://$(find aubo_description)/meshes/aubo_E10_10/collisio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; visual mesh filename=file://$(find aubo_description)/meshes/aubo_E10_10/visual/l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
- link wrist2_Link: geometry collision mesh filename=file://$(find aubo_description)/meshes/aubo_E10_10/collisio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; visual mesh filename=file://$(find aubo_description)/meshes/aubo_E10_10/visual/l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
- link wrist3_Link: geometry collision mesh filename=file://$(find aubo_description)/meshes/aubo_E10_10/collisio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; visual mesh filename=file://$(find aubo_description)/meshes/aubo_E10_10/visual/l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

File: urdf/aubo_E16_10.urdf (robot description, URDF)
Before this commit: robot aubo_E16_10, 8 links, 7 joints
Links:
- link base_link: geometry collision mesh filename=file://$(find aubo_description)/meshes/aubo_E16_10/collisio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; visual mesh filename=file://$(find aubo_description)/meshes/aubo_E16_10/visual/l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
- link foreArm_Link: geometry collision mesh filename=file://$(find aubo_description)/meshes/aubo_E16_10/collisio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; visual mesh filename=file://$(find aubo_description)/meshes/aubo_E16_10/visual/l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
- link shoulder_Link: geometry collision mesh filename=file://$(find aubo_description)/meshes/aubo_E16_10/collisio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; visual mesh filename=file://$(find aubo_description)/meshes/aubo_E16_10/visual/l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
- link upperArm_Link: geometry collision mesh filename=file://$(find aubo_description)/meshes/aubo_E16_10/collisio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; visual mesh filename=file://$(find aubo_description)/meshes/aubo_E16_10/visual/l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
- link wrist1_Link: geometry collision mesh filename=file://$(find aubo_description)/meshes/aubo_E16_10/collisio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; visual mesh filename=file://$(find aubo_description)/meshes/aubo_E16_10/visual/l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
- link wrist2_Link: geometry collision mesh filename=file://$(find aubo_description)/meshes/aubo_E16_10/collisio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; visual mesh filename=file://$(find aubo_description)/meshes/aubo_E16_10/visual/l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
- link wrist3_Link: geometry collision mesh filename=file://$(find aubo_description)/meshes/aubo_E16_10/collisio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; visual mesh filename=file://$(find aubo_description)/meshes/aubo_E16_10/visual/l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

File: urdf/aubo_E20_10.urdf (robot description, URDF)
Before this commit: robot aubo_E20_10, 8 links, 7 joints
Links:
- link base_link: geometry collision mesh filename=file://$(find aubo_description)/meshes/aubo_E20_10/collisio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; visual mesh filename=file://$(find aubo_description)/meshes/aubo_E20_10/visual/l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
- link foreArm_Link: geometry collision mesh filename=file://$(find aubo_description)/meshes/aubo_E20_10/collisio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; visual mesh filename=file://$(find aubo_description)/meshes/aubo_E20_10/visual/l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
- link shoulder_Link: geometry collision mesh filename=file://$(find aubo_description)/meshes/aubo_E20_10/collisio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; visual mesh filename=file://$(find aubo_description)/meshes/aubo_E20_10/visual/l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
- link upperArm_Link: geometry collision mesh filename=file://$(find aubo_description)/meshes/aubo_E20_10/collisio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; visual mesh filename=file://$(find aubo_description)/meshes/aubo_E20_10/visual/l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
- link wrist1_Link: geometry collision mesh filename=file://$(find aubo_description)/meshes/aubo_E20_10/collisio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; visual mesh filename=file://$(find aubo_description)/meshes/aubo_E20_10/visual/l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
- link wrist2_Link: geometry collision mesh filename=file://$(find aubo_description)/meshes/aubo_E20_10/collisio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; visual mesh filename=file://$(find aubo_description)/meshes/aubo_E20_10/visual/l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
- link wrist3_Link: geometry collision mesh filename=file://$(find aubo_description)/meshes/aubo_E20_10/collisio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; visual mesh filename=file://$(find aubo_description)/meshes/aubo_E20_10/visual/l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

File: urdf/aubo_E3.urdf (robot description, URDF)
Before this commit: robot aubo_E3, 8 links, 7 joints
Links:
- link base_link: geometry collision mesh filename=file://$(find aubo_description)/meshes/aubo_E3/collision/li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; visual mesh filename=file://$(find aubo_description)/meshes/aubo_E3/visual/link0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
- link foreArm_Link: geometry collision mesh filename=file://$(find aubo_description)/meshes/aubo_E3/collision/li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; visual mesh filename=file://$(find aubo_description)/meshes/aubo_E3/visual/link3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
- link shoulder_Link: geometry collision mesh filename=file://$(find aubo_description)/meshes/aubo_E3/collision/li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; visual mesh filename=file://$(find aubo_description)/meshes/aubo_E3/visual/link1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
- link upperArm_Link: geometry collision mesh filename=file://$(find aubo_description)/meshes/aubo_E3/collision/li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; visual mesh filename=file://$(find aubo_description)/meshes/aubo_E3/visual/link2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
- link wrist1_Link: geometry collision mesh filename=file://$(find aubo_description)/meshes/aubo_E3/collision/li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; visual mesh filename=file://$(find aubo_description)/meshes/aubo_E3/visual/link4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
- link wrist2_Link: geometry collision mesh filename=file://$(find aubo_description)/meshes/aubo_E3/collision/li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; visual mesh filename=file://$(find aubo_description)/meshes/aubo_E3/visual/link5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
- link wrist3_Link: geometry collision mesh filename=file://$(find aubo_description)/meshes/aubo_E3/collision/li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; visual mesh filename=file://$(find aubo_description)/meshes/aubo_E3/visual/link6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

File: urdf/aubo_E3_10.urdf (robot description, URDF)
Before this commit: robot aubo_e3_10, 8 links, 7 joints
Links:
- link base_link: geometry collision mesh filename=file://$(find aubo_description)/meshes/aubo_e3_10/collision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; visual mesh filename=file://$(find aubo_description)/meshes/aubo_e3_10/visual/li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
- link foreArm_Link: geometry collision mesh filename=file://$(find aubo_description)/meshes/aubo_e3_10/collision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; visual mesh filename=file://$(find aubo_description)/meshes/aubo_e3_10/visual/li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
- link shoulder_Link: geometry collision mesh filename=file://$(find aubo_description)/meshes/aubo_e3_10/collision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; visual mesh filename=file://$(find aubo_description)/meshes/aubo_e3_10/visual/li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
- link upperArm_Link: geometry collision mesh filename=file://$(find aubo_description)/meshes/aubo_e3_10/collision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; visual mesh filename=file://$(find aubo_description)/meshes/aubo_e3_10/visual/li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
- link wrist1_Link: geometry collision mesh filename=file://$(find aubo_description)/meshes/aubo_e3_10/collision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; visual mesh filename=file://$(find aubo_description)/meshes/aubo_e3_10/visual/li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
- link wrist2_Link: geometry collision mesh filename=file://$(find aubo_description)/meshes/aubo_e3_10/collision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; visual mesh filename=file://$(find aubo_description)/meshes/aubo_e3_10/visual/li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
- link wrist3_Link: geometry collision mesh filename=file://$(find aubo_description)/meshes/aubo_e3_10/collision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; visual mesh filename=file://$(find aubo_description)/meshes/aubo_e3_10/visual/li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
