Commit message: Change description to be comppatible with ROS2 jazzy

File: urdf/aubo_E5_10.urdf (robot description, URDF)
Before this commit: robot aubo_E5_10, 8 links, 7 joints
Links:
- link base_link: geometry collision mesh filename=file://$(find aubo_description)/meshes/aubo_E5_10/collision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; visual mesh filename=file://$(find aubo_description)/meshes/aubo_E5_10/visual/li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
- link foreArm_Link: geometry collision mesh filename=file://$(find aubo_description)/meshes/aubo_E5_10/collision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; visual mesh filename=file://$(find aubo_description)/meshes/aubo_E5_10/visual/li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
- link shoulder_Link: geometry collision mesh filename=file://$(find aubo_description)/meshes/aubo_E5_10/collision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; visual mesh filename=file://$(find aubo_description)/meshes/aubo_E5_10/visual/li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
- link upperArm_Link: geometry collision mesh filename=file://$(find aubo_description)/meshes/aubo_E5_10/collision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; visual mesh filename=file://$(find aubo_description)/meshes/aubo_E5_10/visual/li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
- link wrist1_Link: geometry collision mesh filename=file://$(find aubo_description)/meshes/aubo_E5_10/collision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; visual mesh filename=file://$(find aubo_description)/meshes/aubo_E5_10/visual/li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
- link wrist2_Link: geometry collision mesh filename=file://$(find aubo_description)/meshes/aubo_E5_10/collision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; visual mesh filename=file://$(find aubo_description)/meshes/aubo_E5_10/visual/li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
- link wrist3_Link: geometry collision mesh filename=file://$(find aubo_description)/meshes/aubo_E5_10/collision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; visual mesh filename=file://$(find aubo_description)/meshes/aubo_E5_10/visual/li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

File: urdf/aubo_ES3.urdf (robot description, URDF)
Before this commit: robot aubo_ES3, 8 links, 7 joints
Links:
- link base_link: geometry collision mesh filename=file://$(find aubo_description)/meshes/aubo_ES3/collision/l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; visual mesh filename=file://$(find aubo_description)/meshes/aubo_ES3/visual/link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
- link foreArm_Link: geometry collision mesh filename=file://$(find aubo_description)/meshes/aubo_ES3/collision/l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; visual mesh filename=file://$(find aubo_description)/meshes/aubo_ES3/visual/link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
- link shoulder_Link: geometry collision mesh filename=file://$(find aubo_description)/meshes/aubo_ES3/collision/l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; visual mesh filename=file://$(find aubo_description)/meshes/aubo_ES3/visual/link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
- link upperArm_Link: geometry collision mesh filename=file://$(find aubo_description)/meshes/aubo_ES3/collision/l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; visual mesh filename=file://$(find aubo_description)/meshes/aubo_ES3/visual/link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
- link wrist1_Link: geometry collision mesh filename=file://$(find aubo_description)/meshes/aubo_ES3/collision/l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; visual mesh filename=file://$(find aubo_description)/meshes/aubo_ES3/visual/link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
- link wrist2_Link: geometry collision mesh filename=file://$(find aubo_description)/meshes/aubo_ES3/collision/l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; visual mesh filename=file://$(find aubo_description)/meshes/aubo_ES3/visual/link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
- link wrist3_Link: geometry collision mesh filename=file://$(find aubo_description)/meshes/aubo_ES3/collision/l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; visual mesh filename=file://$(find aubo_description)/meshes/aubo_ES3/visual/link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

File: urdf/aubo_ES5.urdf (robot description, URDF)
Before this commit: robot aubo_ES5, 8 links, 7 joints
Links:
- link base_link: geometry collision mesh filename=file://$(find aubo_description)/meshes/aubo_ES5/collision/l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; visual mesh filename=file://$(find aubo_description)/meshes/aubo_ES5/visual/link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
- link foreArm_Link: geometry collision mesh filename=file://$(find aubo_description)/meshes/aubo_ES5/collision/l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; visual mesh filename=file://$(find aubo_description)/meshes/aubo_ES5/visual/link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
- link shoulder_Link: geometry collision mesh filename=file://$(find aubo_description)/meshes/aubo_ES5/collision/l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; visual mesh filename=file://$(find aubo_description)/meshes/aubo_ES5/visual/link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
- link upperArm_Link: geometry collision mesh filename=file://$(find aubo_description)/meshes/aubo_ES5/collision/l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; visual mesh filename=file://$(find aubo_description)/meshes/aubo_ES5/visual/link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
- link wrist1_Link: geometry collision mesh filename=file://$(find aubo_description)/meshes/aubo_ES5/collision/l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; visual mesh filename=file://$(find aubo_description)/meshes/aubo_ES5/visual/link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
- link wrist2_Link: geometry collision mesh filename=file://$(find aubo_description)/meshes/aubo_ES5/collision/l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; visual mesh filename=file://$(find aubo_description)/meshes/aubo_ES5/visual/link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
- link wrist3_Link: geometry collision mesh filename=file://$(find aubo_description)/meshes/aubo_ES5/collision/l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; visual mesh filename=file://$(find aubo_description)/meshes/aubo_ES5/visual/link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

File: urdf/aubo_ES5_B0.urdf (robot description, URDF)
Before this commit: robot aubo_ES5_B0, 8 links, 7 joints
Links:
- link base_link: geometry collision mesh filename=file://$(find aubo_description)/meshes/aubo_ES5_B0/collisio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; visual mesh filename=file://$(find aubo_description)/meshes/aubo_ES5_B0/visual/l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
- link foreArm_Link: geometry collision mesh filename=file://$(find aubo_description)/meshes/aubo_ES5_B0/collisio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; visual mesh filename=file://$(find aubo_description)/meshes/aubo_ES5_B0/visual/l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
- link shoulder_Link: geometry collision mesh filename=file://$(find aubo_description)/meshes/aubo_ES5_B0/collisio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; visual mesh filename=file://$(find aubo_description)/meshes/aubo_ES5_B0/visual/l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
- link upperArm_Link: geometry collision mesh filename=file://$(find aubo_description)/meshes/aubo_ES5_B0/collisio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; visual mesh filename=file://$(find aubo_description)/meshes/aubo_ES5_B0/visual/l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
- link wrist1_Link: geometry collision mesh filename=file://$(find aubo_description)/meshes/aubo_ES5_B0/collisio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; visual mesh filename=file://$(find aubo_description)/meshes/aubo_ES5_B0/visual/l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
- link wrist2_Link: geometry collision mesh filename=file://$(find aubo_description)/meshes/aubo_ES5_B0/collisio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; visual mesh filename=file://$(find aubo_description)/meshes/aubo_ES5_B0/visual/l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
- link wrist3_Link: geometry collision mesh filename=file://$(find aubo_description)/meshes/aubo_ES5_B0/collisio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; visual mesh filename=file://$(find aubo_description)/meshes/aubo_ES5_B0/visual/l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

File: urdf/aubo_ES5_B1.urdf (robot description, URDF)
Before this commit: robot aubo_ES5_B1, 8 links, 7 joints
Links:
- link base_link: geometry collision mesh filename=file://$(find aubo_description)/meshes/aubo_ES5_B1/collisio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; visual mesh filename=file://$(find aubo_description)/meshes/aubo_ES5_B1/visual/l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
- link foreArm_Link: geometry collision mesh filename=file://$(find aubo_description)/meshes/aubo_ES5_B1/collisio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; visual mesh filename=file://$(find aubo_description)/meshes/aubo_ES5_B1/visual/l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
- link shoulder_Link: geometry collision mesh filename=file://$(find aubo_description)/meshes/aubo_ES5_B1/collisio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; visual mesh filename=file://$(find aubo_description)/meshes/aubo_ES5_B1/visual/l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
- link upperArm_Link: geometry collision mesh filename=file://$(find aubo_description)/meshes/aubo_ES5_B1/collisio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; visual mesh filename=file://$(find aubo_description)/meshes/aubo_ES5_B1/visual/l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
- link wrist1_Link: geometry collision mesh filename=file://$(find aubo_description)/meshes/aubo_ES5_B1/collisio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; visual mesh filename=file://$(find aubo_description)/meshes/aubo_ES5_B1/visual/l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
- link wrist2_Link: geometry collision mesh filename=file://$(find aubo_description)/meshes/aubo_ES5_B1/collisio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; visual mesh filename=file://$(find aubo_description)/meshes/aubo_ES5_B1/visual/l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
- link wrist3_Link: geometry collision mesh filename=file://$(find aubo_description)/meshes/aubo_ES5_B1/collisio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; visual mesh filename=file://$(find aubo_description)/meshes/aubo_ES5_B1/visual/l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
