Commit message: Modify end effector

File: urdf/xacro/inc/aubo_ros2_macro.xacro (robot description, xacro)
@@ -6,13 +6,19 @@
       <parent link="wrist3_Link" />
       <child link ="ee_link" />
-      <origin xyz="0.0 0.0 0.0" rpy="0.0 0.0 ${pi/2.0}" />
+      <origin xyz="0.0 0.0 0.2" rpy="0.0 0.0 0.0" />
     </joint>
     <link name="ee_link">
       <collision>
         <geometry>
-          <box size="0.01 0.01 0.01"/>
+          <box size="0.1 0.1 0.2"/>
         </geometry>
-        <origin rpy="0 0 0" xyz="-0.01 0 0"/>
+        <origin rpy="0 0 0" xyz="-0.1 0 0"/>
       </collision>
+      <visual>
+        <geometry>
+          <box size="0.1 0.1 0.2"/>
+        </geometry>
+        <origin rpy="0 0 0" xyz="-0.1 0 0"/>
+      </visual>
     </link>
     <transmission name="shoulder_trans">

Commit message: Adjust end effector

File: urdf/xacro/inc/aubo_ros2_macro.xacro (robot description, xacro)
@@ -11,13 +11,13 @@
       <collision>
         <geometry>
-          <box size="0.1 0.1 0.2"/>
+          <box size="0.1 0.1 0.16"/>
         </geometry>
-        <origin rpy="0 0 0" xyz="-0.1 0 0"/>
+        <origin rpy="0 0 0" xyz="0 0 -0.12"/>
       </collision>
       <visual>
         <geometry>
-          <box size="0.1 0.1 0.2"/>
+          <box size="0.1 0.1 0.16"/>
         </geometry>
-        <origin rpy="0 0 0" xyz="-0.1 0 0"/>
+        <origin rpy="0 0 0" xyz="0 0 -0.12"/>
       </visual>
     </link>
